File: Hardware/SparkFun_MicroSD_Sniffer.brd (EAGLE design)
At the start: 47 x 27.9 mm, 9 parts, among them U1 MICRO-SDCARD, U2 microSD Socket

Commit message: changed schematic and board design
Parts:
- removed FID1, FID2: FIDUCIAL1X2, SparkFun-Aesthetics:FIDUCIAL-1X2
- removed FRAME1: (no value), SparkFun-Aesthetics:CREATIVE_COMMONS
- removed LOGO1: OSHW-LOGOM, SparkFun-Aesthetics:OSHW-LOGO-M
- removed LOGO2: SFE_LOGO_FLAME.2_INCH, SparkFun-Aesthetics:SFE_LOGO_FLAME_.2
- removed LOGO3: SFE_LOGO_NAME_FLAME.1_INCH, SparkFun-Aesthetics:SFE_LOGO_NAME_FLAME_.1
- removed U2: microSD Socket, SparkFun-Connectors:MICROSD_1:1
- JP1: device SparkFun:1X08 -> pinhead:2X04
- U1: value MICRO-SDCARD -> SPARKFUN_MICRO-SDCARD; device SparkFun-Boards:MICRO-SDCARD -> microsniffer-v14:SPARKFUN_MICRO-SDCARD
- moved JP1 26.4 mm to (26.5, 12.7), turned to 270 degrees
- moved U1 0.15 mm to (47.0, 7.75)
Connections:
- net CD/DAT3: now also JP1.8; no longer JP1.2, U2.2
- net CLK: now also JP1.3; no longer JP1.6, U2.5
- net CMD: now also JP1.5; no longer JP1.3, U2.3
- net DAT0: now also JP1.1; no longer JP1.7, U2.7
- net DAT1: now also JP1.2; no longer JP1.8, U2.8
- net DAT2: now also JP1.7; no longer JP1.1, U2.1
- net GND: no longer U2.6, U2.CD1, U2.CD2, U2.GND1, U2.GND3
- net VCC: now also JP1.6; no longer JP1.5, U2.4
Routing:
- net DAT2: track 68.5 -> 20.6 mm
- net CD/DAT3: track 62.4 -> 17.5 mm, vias 1 -> 0
- net CMD: track 59.6 -> 20.5 mm, vias 1 -> 0
- net DAT1: track 50.6 -> 17.1 mm, vias 1 -> 0
- net VCC: track 54.0 -> 21.6 mm, vias 1 -> 0
- net CLK: track 52.2 -> 20.3 mm, vias 1 -> 0
- net DAT0: track 50.8 -> 20.2 mm, vias 1 -> 0
- net GND: track 0.00 -> 20.9 mm, vias 2 -> 0
- removed copper zone on layer 1, net GND
- removed copper zone on layer 16, net GND
Other:
- board size 47 x 27.9 mm -> 23.1 x 10.9 mm
- board text added: "DAT3"
- board text removed: "CD"
- board text removed: "PCB must be no thicker than 0.75mm"
- board text removed: "Revised by: Patrick Alberts"
- board text removed: "Tim Holmberg"
- board text removed: "V10"
- board text removed: "microSD Sniffer"
